File: PCB/measuring-sending-module/outside-entrance-controller.kicad_pcb (KiCad board)
At the start: 2 copper layers, 80 x 72.4 mm, 71 parts, among them J1 ICP, J2 Power-Supply-12V, J3 Conn_01x03, J4 Gate-SW, J5 Screw_Terminal_01x10, Q1 BC547, Q2 BC547, Q3 BC547, U1 L7805, U2 PIC16F819-ISO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

Commit message: Receiver and transmiter code update, PCB and schematic update
Parts:
- moved C10 6.25 mm to (202.2, 115.3)
Connections:
- C10 pad 1: +5V -> +12V
- J3 pad 1: /RA0 -> Net-(J3-Pad1)
- J3 pad 2: /RA7 -> Net-(J3-Pad2)
- J3 pad 3: /RA6 -> Net-(J3-Pad3)
- U3 pad 2: +5V -> +12V
Routing:
- net +12V: track 105.9 -> 155.4 mm, vias 0 -> 2
- net +5V: track 209.2 -> 203.9 mm
- net GND: track 78.6 -> 79.9 mm

Commit message: update
Parts:
- added Q4: BC807, TO_SOT_Packages_SMD:SOT-23, F.Cu at (208.2, 110.4)
- added Q5: BC817, TO_SOT_Packages_SMD:SOT-23, F.Cu at (208.0, 113.9)
- added R25: 4k7, Resistors_SMD:R_0805_HandSoldering, F.Cu at (207.5, 102.7)
- added R26: 10k, Resistors_SMD:R_0805_HandSoldering, F.Cu at (205.4, 102.7)
- added R27: 10k, Resistors_SMD:R_0805_HandSoldering, F.Cu at (205.1, 113.2)
- J3: value Conn_01x03 -> Conn_01x02; footprint Pin_Headers:Pin_Header_Straight_1x03_Pitch2.54mm -> Pin_Headers:Pin_Header_Straight_1x02_Pitch2.54mm
- moved J3 5.08 mm to (182.6, 101.9), turned to 0 degrees
Connections:
- J3 pad 1: Net-(J3-Pad1) -> /RA6
- J3 pad 2: Net-(J3-Pad2) -> /RA7
- U2 pad 17: /RA0 -> /radio_en
- U3 pad 2: +12V -> Net-(Q4-Pad3)
Routing:
- net /radio_en: track 0.00 -> 19.9 mm
- net /RA0: track 19.9 -> 0.00 mm
